Commit message: test1

File: uav_simulator/Utils/testbot_description/urdf/test.urdf (robot description, URDF)
Before this commit: robot myfirst, 1 links, 0 joints
Links:
- added link camera_link
Joints:
- added joint depth_camera_joint: type fixed, parent base_link, child camera_link, origin xyz=0.1 0 0 rpy=-1.5 0 1.5
